File: MPHS.brd (EAGLE design)
At the start: 25.4 x 34.3 mm, 22 parts, among them U1 SPI_FLASH-X25XXSMD, U2 MCP1701, U3 RFM69W

Commit message: New photo with LED installed (parts arrived)
Changed board layout and schematic to have proper LED component.  No
change to actual BOM or circuit.  Shot new photo of board with LED
installed.
Parts:
- removed D1: LED, SparkFun-Resistors:0805
- added LED1: LED-0805, ChipsParts:0805-LED
Connections:
- net N$13: now also LED1.A; no longer D1.2
- net N$15: now also LED1.C; no longer D1.1
Changed lines of the file:
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@@
 <text x="24.13" y="3.4925" size="0.8128" layer="21" font="vector" ratio="15" align="bottom-center">3V3</text>
 <text x="19.3675" y="5.08" size="0.8128" layer="21" font="vector" ratio="15" rot="R90" align="bottom-center">FSEL</text>
-<wire x1="15.875" y1="6.0325" x2="16.51" y2="6.0325" width="0.127" layer="21"/>
-<wire x1="16.51" y1="6.0325" x2="17.145" y2="6.0325" width="0.127" layer="21"/>
-<wire x1="16.51" y1="6.0325" x2="15.875" y2="5.3975" width="0.127" layer="21"/>
-<wire x1="16.51" y1="6.0325" x2="17.145" y2="5.3975" width="0.127" layer="21"/>
 </plain>
 <attributes>
@@
 </element>
 <element name="JP1" library="SparkFun-Connectors" package="1X10" value="M10&quot;" x="1.27" y="1.905" smashed="yes"/>
-<element name="D1" library="SparkFun-Resistors" package="0805" value="LED" x="16.51" y="5.715" smashed="yes" rot="R270">
-<attribute name="NAME" x="17.3355" y="6.477" size="0.4064" layer="25" ratio="15" rot="R270"/>
-<attribute name="VALUE" x="15.113" y="6.731" size="0.4064" layer="27" rot="R270"/>
+<element name="LED1" library="ChipsParts" package="0805-LED" value="LED-0805" x="16.51" y="5.715" smashed="yes" rot="R90">
+<attribute name="NAME" x="15.6845" y="4.953" size="0.4064" layer="25" ratio="15" rot="R90"/>
+<attribute name="VALUE" x="17.907" y="4.699" size="0.4064" layer="27" rot="R90"/>
 </element>
 </elements>
@@
 <signal name="N$13">
 <contactref element="JP1" pad="7"/>
-<contactref element="D1" pad="2"/>
-<wire x1="16.51" y1="1.905" x2="16.51" y2="4.815" width="0.254" layer="1"/>
+<contactref element="LED1" pad="A"/>
+<wire x1="16.51" y1="4.815" x2="16.51" y2="1.905" width="0.254" layer="1"/>
 </signal>
 <signal name="N$15">
 <contactref element="R7" pad="2"/>
-<contactref element="D1" pad="1"/>
-<wire x1="16.51" y1="6.615" x2="17.515" y2="6.615" width="0.254" layer="1"/>
 <wire x1="17.515" y1="6.615" x2="18.415" y2="5.715" width="0.254" layer="1"/>
 <wire x1="18.415" y1="5.715" x2="20.055" y2="5.715" width="0.254" layer="1"/>
+<contactref element="LED1" pad="C"/>
+<wire x1="16.51" y1="6.615" x2="17.515" y2="6.615" width="0.254" layer="1"/>
 </signal>
 </signals>
