File: MPHS-RFM69C.brd (EAGLE design)
At the start: 25.4 x 34.3 mm, 22 parts, among them U1 SPI_FLASH-X25XXSMD, U2 MCP1701

Commit message: Changed VReg to 1117
Parts:
- removed U2: MCP1701, ChipsParts:SOT-89
- added U3: (no value), SparkFun-PowerIC:SOT223
- moved C3 1.80 mm to (22.9, 14.0), turned to 90 degrees
- moved C2 1.27 mm to (22.9, 10.2), turned to 270 degrees
Connections:
- net GND: now also U3.1; no longer U2.1
- net N$2: now also U3.3; no longer U2.2
- net VCC: now also U3.2, U3.4; no longer U2.3
Routing:
- net GND: track 12.6 -> 6.35 mm, vias 7 -> 5
- net N$2: track 26.8 -> 30.6 mm
- net VCC: track 59.5 -> 62.0 mm
- net N$14: track 19.6 -> 22.0 mm
Other:
- board text added: "C.Schnarel 04OCT2015"
- board text removed: "C.Schnarel 02OCT2015"
